Commit message: update urdf

File: jetbot_description/urdf/jetbot.xacro (robot description, xacro)
@@ -139,5 +139,5 @@
             <origin xyz="0.0 0.0 0.0" rpy="0.0 0.0 0.0"/>
             <geometry>
-                <cylinder radius="0.035" length="0.02"/>
+                <cylinder radius="0.035" length="0.06"/>
             </geometry>
             <material name="">
@@ -170,5 +170,4 @@
             <box size="0.02 0.02 0.02"/>
         </geometry>
-        <material name="orange"/>
         </visual>
         <inertial>
@@ -182,5 +181,5 @@
     </link>
     <joint name="imu_joint" type="fixed">
-        <origin xyz="0.0 0.0 0.0" rpy="0.0 0.0 0.0"/>
+        <origin xyz="-0.1 0.0 0.0" rpy="0.0 0.0 0.0"/>
         <parent link="base_link"/>
         <child link="imu_link"/>
